File: PiPX4.kicad_pcb (KiCad board)
At the start: 4 copper layers, 29 x 44.7 mm, 105 parts, among them J1 Conn_01x04_MountingPin, J2 Conn_01x04_MountingPin, J3 Conn_01x04_MountingPin, J4 USB_C_Receptacle, SW1 SW_Push, U1 MKDV4GCL-AB, U2 V3S-ALLWINNER, U3 EA3036, U4 GW1N_LV4QN32C6/I5, U5 HMC5883L-TR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

Commit message: add teardrop, change the size of drill to 0.45mm
Signed-off-by: ncerzzk <huangzzk@bupt.edu.cn>
Routing:
- net +3V3: track 175.0 -> 171.4 mm
- net /V3s_core/SD_DATA1: track 13.3 -> 14.6 mm
Other:
- board text added: "TMS"

Commit message: edit spacing to 0.999mm because of JLC
Signed-off-by: ncerzzk <huangzzk@bupt.edu.cn>
Routing:
- net +3V3: track 171.4 -> 159.7 mm, vias 22 -> 23
- net GND: track 58.9 -> 56.8 mm, vias 32 -> 31
- net Net-(C15-Pad2): track 3.31 -> 4.64 mm, vias 1 -> 2
- net /FPGA/FPGA_CTL1: track 11.7 -> 10.3 mm
- net /FPGA/FPGA_CTL2: track 11.7 -> 11.1 mm

Commit message: fix u0_rx u0_tx wrong connection issue, fix the hole in V3s GND PAD is too small issue. update to V0.95.
Signed-off-by: ncerzzk <huangzzk@bupt.edu.cn>
Connections:
- U2 pad 48: /U0_RX -> /U0_TX
- U2 pad 49: /U0_TX -> /U0_RX
Routing:
- net +3V3: track 159.7 -> 158.3 mm, vias 23 -> 22
- net /FPGAIO7: track 0.74 -> 0.00 mm, vias 1 -> 0
Other:
- board text added: "PiPX4-V3s V0.95"
- board text removed: "PiPX4-V3s V0.9"
