File: AutoPilotPi.kicad_pcb (KiCad board)
At the start: 4 copper layers, 29 x 44.7 mm, 105 parts, among them J1 Conn_01x04_MountingPin, J2 Conn_01x04_MountingPin, J3 Conn_01x04_MountingPin, J4 USB_C_Receptacle, SW1 SW_Push, U1 MKDV4GCL-AB, U2 V3S-ALLWINNER, U3 EA3036, U4 GW1N_LV4QN32C6/I5, U5 HMC5883L-TR, U6 SPL06-001, U7 v3s_flight_controller, U8 TLV71312PDBV, Y1 Crystal, Y2 Crystal_GND24_Small

Commit message: update mini
Signed-off-by: huangzzk <huangcmzzk@gmail.com>
Parts:
- removed SW1: SW_Push, Button_Switch_SMD:SW_Push_SPST_NO_Alps_SKRK
- removed U7: v3s_flight_controller, ic_footprint:Flight_Core
- added C57: 10u, Capacitor_SMD:C_0603_1608Metric, F.Cu at (77.1, 71.5)
- added C58: 10u, Capacitor_SMD:C_0603_1608Metric, F.Cu at (78.8, 71.5)
- added C59: 1u, Capacitor_SMD:C_0402_1005Metric, F.Cu at (72.9, 83.6)
- added C60: 0.1u, Capacitor_SMD:C_0402_1005Metric, F.Cu at (72.9, 82.4)
- added D4: LED, LED_SMD:LED_0603_1608Metric, F.Cu at (74.8, 83.3)
- added J5: Conn_01x03, Connector_Molex:Molex_CLIK-Mate_502386-0370_1x03-1MP_P1.25mm_Horizontal, B.Cu at (99.1, 88.1)
- added J6: Conn_01x03, Connector_Molex:Molex_CLIK-Mate_502386-0370_1x03-1MP_P1.25mm_Horizontal, F.Cu at (77.2, 88.2)
- added J7: Conn_01x03, Connector_Molex:Molex_CLIK-Mate_502386-0370_1x03-1MP_P1.25mm_Horizontal, F.Cu at (99.2, 87.5)
- added L1: L, Inductor_SMD:L_Abracon_ASPI-3012S, F.Cu at (74.0, 71.6)
- added M1: xr819, ic_footprint:xr819_module, B.Cu at (84.5, 44.9)
- added M2: mini_elrs, ic_footprint:mini_elrs, F.Cu at (84.9, 38.2)
- added Q1: Q_NMOS_GSD, Package_TO_SOT_SMD:SOT-23, B.Cu at (74.6, 82.3)
- added Q2: Q_NMOS_GSD, Package_TO_SOT_SMD:SOT-23, B.Cu at (95.5, 82.4)
- added R17: 0R, Resistor_SMD:R_0402_1005Metric, F.Cu at (93.5, 86.9)
- added R28: 10K, Resistor_SMD:R_0402_1005Metric, B.Cu at (75.4, 79.8)
- added R29: 10K, Resistor_SMD:R_0402_1005Metric, B.Cu at (99.7, 84.1)
- added U9: ETA9640, Package_SO:SOIC-8-1EP_3.9x4.9mm_P1.27mm_EP2.41x3.3mm, F.Cu at (75.5, 77.5)
- C11, C12, C17, C18: value 18pf -> 18p
- C15: value 1uF -> 1u
- C31, C34: value 4.7uF -> 4.7u
- C51: value 0.22uF -> 0.22u
- J2: value Conn_01x04_MountingPin -> Conn_01x03; footprint Connector_Molex:Molex_CLIK-Mate_502382-0470_1x04-1MP_P1.25mm_Vertical -> Connector_Molex:Molex_CLIK-Mate_502386-0370_1x03-1MP_P1.25mm_Horizontal
- J3: value Conn_01x04_MountingPin -> Conn_01x02; footprint Connector_Molex:Molex_CLIK-Mate_502382-0470_1x04-1MP_P1.25mm_Vertical -> Connector_PinHeader_2.54mm:PinHeader_1x02_P2.54mm_Vertical; moved to F.Cu
- R20: value 0R -> 1.2k; moved to F.Cu
- R21: value 10K -> 0R
- R23: value 4.7k -> 4.7K
- R27: value 499R -> 10K; moved to F.Cu
- U8: value TLV71312PDBV -> ME6212C12M5G
- moved J2 39.3 mm to (77.0, 88.2)
- moved R20 30.0 mm to (77.6, 82.9), turned to -90 degrees
- moved R27 26.6 mm to (76.2, 82.9), turned to 90 degrees
- moved J3 22.4 mm to (75.2, 68.2), turned to 90 degrees
- moved J4 15.1 mm to (76.3, 61.1), turned to -90 degrees
- moved J1 10.3 mm to (87.2, 87.8)
Connections:
- J2 pad 1: +5V -> /FPGAIO5
- J2 pad 2: /U1_TX -> +BATT
- J2 pad 3: /U1_RX -> Net-(Q1-Pad3)
- J2 pad MP: GND -> (no net)
- J3 pad 1: +5V -> +BATT
- J3 pad 2: /U2_TX -> GNDPWR
- R20 pad 1: +5V -> Net-(R20-Pad1)
- R20 pad 2: VBUS -> GND
- R27 pad 2: GND -> Net-(R27-Pad2)
- U2 pad 6: unconnected-(U2-Pad6) -> /WIRQ
- U2 pad 7: unconnected-(U2-Pad7) -> /WREST
Routing:
- net GNDPWR: track 0.00 -> 76.4 mm, vias 0 -> 13
- net +BATT: track 0.00 -> 65.9 mm, vias 0 -> 2
- net +3V3: track 159.9 -> 203.9 mm, vias 21 -> 25
- net /U2_TX: track 32.1 -> 0.00 mm, vias 3 -> 0
- net /U2_RX: track 31.6 -> 0.00 mm, vias 2 -> 0
- net /FPGAIO7: track 0.00 -> 27.3 mm, vias 0 -> 3
- net /WIRQ: track 0.00 -> 26.8 mm, vias 0 -> 2
- net /FPGAIO8: track 25.3 -> 0.00 mm, vias 1 -> 0
- net (no net): track 0.00 -> 24.8 mm
- net +1V8: track 63.9 -> 87.0 mm
- net /FPGAIO6: track 22.4 -> 0.00 mm, vias 2 -> 0
- net /FPGAIO9: track 22.4 -> 0.00 mm, vias 1 -> 0
- net /FPGAIO0: track 21.1 -> 0.00 mm, vias 1 -> 0
- net /FPGAIO4: track 20.0 -> 0.00 mm, vias 1 -> 0
- net /FPGAIO2: track 19.5 -> 0.00 mm, vias 1 -> 0
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- removed copper zone on In2.Cu, net GND
Other:
- board size 29 x 44.7 mm -> 32.9 x 59.2 mm
- board text added: "-"
- board text added: "BAT"
- board text removed: "AutoPilotPi V0.97"
- board text removed: "CLK"
- board text removed: "CMD"
- board text removed: "CSN"
- board text removed: "D0"
- board text removed: "D1"
- board text removed: "D2"
- board text removed: "D3"
- board text removed: "GND"
- board text removed: "IO1"
- board text removed: "IO2"
- board text removed: "IO3"
- board text removed: "IO4"
- board text removed: "IO5"
- board text removed: "IO6"
- board text removed: "IO8"
- board text removed: "IO9"
- board text removed: "MISO"
- board text removed: "MOSI"
- board text removed: "SCL"
- board text removed: "SCLK"
- board text removed: "SDA"
- board text removed: "TCK"
- board text removed: "TDI"
- board text removed: "TDO"
- board text removed: "TMS"
- board text removed: "U2"
- board text removed: "X"
- board text removed: "Y"

Commit message: temply update
Signed-off-by: ncerzzk <huangzzk@bupt.edu.cn>
Parts:
- removed C57, C58: 10u, Capacitor_SMD:C_0603_1608Metric
- removed C59: 1u, Capacitor_SMD:C_0402_1005Metric
- removed C60: 0.1u, Capacitor_SMD:C_0402_1005Metric
- removed D4: LED, LED_SMD:LED_0603_1608Metric
- removed Q1, Q2: Q_NMOS_GSD, Package_TO_SOT_SMD:SOT-23
- removed U9: ETA9640, Package_SO:SOIC-8-1EP_3.9x4.9mm_P1.27mm_EP2.41x3.3mm
- added J10: Conn_01x03, Connector_Molex:Molex_PicoBlade_53047-0310_1x03_P1.25mm_Vertical, F.Cu at (10.9, 68.7)
- added J11: Conn_01x03, Connector_Molex:Molex_PicoBlade_53047-0310_1x03_P1.25mm_Vertical, F.Cu at (6.23, 68.7)
- added J12: Conn_01x03, Connector_Molex:Molex_PicoBlade_53047-0310_1x03_P1.25mm_Vertical, F.Cu at (41.4, 74.2)
- added J13: Conn_01x03, Connector_Molex:Molex_PicoBlade_53047-0310_1x03_P1.25mm_Vertical, F.Cu at (34.6, 74.1)
- added J14: Conn_01x03, Connector_Molex:Molex_PicoBlade_53047-0310_1x03_P1.25mm_Vertical, F.Cu at (40.9, 68.7)
- added J15: Conn_01x03, Connector_Molex:Molex_PicoBlade_53047-0310_1x03_P1.25mm_Vertical, F.Cu at (33.8, 69.3)
- added J16: Conn_01x04_MountingPin, Connector_Molex:Molex_CLIK-Mate_502382-0470_1x04-1MP_P1.25mm_Vertical, F.Cu at (39.6, 59.2)
- added J17: Conn_01x04_MountingPin, Connector_Molex:Molex_CLIK-Mate_502382-0470_1x04-1MP_P1.25mm_Vertical, F.Cu at (25.7, 59.2)
- added J18: USB_C_Receptacle, Connector_USB:USB_C_Receptacle_Palconn_UTC16-G, F.Cu at (9.70, 48.0)
- added J8: Conn_01x03, Connector_PinHeader_2.54mm:PinHeader_1x03_P2.54mm_Vertical, F.Cu at (96.5, 93.0)
- added J9: Conn_01x03, Connector_PinHeader_2.54mm:PinHeader_1x03_P2.54mm_Vertical, F.Cu at (94.0, 93.0)
- added R30: 10K, Resistor_SMD:R_0402_1005Metric, F.Cu at (14.1, 79.1)
- added R31: 0R, Resistor_SMD:R_0402_1005Metric, F.Cu at (8.27, 81.0)
- added R32: 0R, Resistor_SMD:R_0402_1005Metric, F.Cu at (11.2, 79.1)
- added R33: NC, Resistor_SMD:R_0402_1005Metric, F.Cu at (17.0, 83.0)
- added R34: NC, Resistor_SMD:R_0402_1005Metric, F.Cu at (19.9, 81.0)
- added R35: 0R, Resistor_SMD:R_0402_1005Metric, F.Cu at (19.9, 77.1)
- added R36: 0R, Resistor_SMD:R_0402_1005Metric, F.Cu at (14.1, 81.0)
- added R37: NC, Resistor_SMD:R_0402_1005Metric, F.Cu at (5.36, 83.0)
- added R38: NC, Resistor_SMD:R_0402_1005Metric, F.Cu at (17.0, 81.0)
- added R39: 0R, Resistor_SMD:R_0402_1005Metric, F.Cu at (5.36, 81.0)
- added R40: 0R, Resistor_SMD:R_0402_1005Metric, F.Cu at (11.2, 81.0)
- added R41: NC, Resistor_SMD:R_0402_1005Metric, F.Cu at (5.36, 79.1)
- added R42: 0R, Resistor_SMD:R_0402_1005Metric, F.Cu at (8.27, 83.0)
- added R43: NC, Resistor_SMD:R_0402_1005Metric, F.Cu at (14.1, 83.0)
- added R44: 0R, Resistor_SMD:R_0402_1005Metric, F.Cu at (14.1, 77.1)
- added R45: NC, Resistor_SMD:R_0402_1005Metric, F.Cu at (17.0, 77.1)
- added R46: NC, Resistor_SMD:R_0402_1005Metric, F.Cu at (8.27, 77.1)
- added R47: 0R, Resistor_SMD:R_0402_1005Metric, F.Cu at (19.9, 79.1)
- added R48: 0R, Resistor_SMD:R_0402_1005Metric, F.Cu at (17.0, 79.1)
- added R49: NC, Resistor_SMD:R_0402_1005Metric, F.Cu at (23.6, 69.8)
- added R50: NC, Resistor_SMD:R_0402_1005Metric, F.Cu at (5.36, 77.1)
- added R51: 0R, Resistor_SMD:R_0402_1005Metric, F.Cu at (11.2, 77.1)
- added R52: 0R, Resistor_SMD:R_0402_1005Metric, F.Cu at (11.2, 83.0)
- added R53: NC, Resistor_SMD:R_0402_1005Metric, F.Cu at (22.8, 77.1)
- added R54: NC, Resistor_SMD:R_0402_1005Metric, F.Cu at (8.27, 79.1)
- added R55: 0R, Resistor_SMD:R_0402_1005Metric, F.Cu at (27.4, 46.9)
- added R56: NC, Resistor_SMD:R_0402_1005Metric, F.Cu at (18.8, 53.2)
- added R57: 0R, Resistor_SMD:R_0402_1005Metric, F.Cu at (18.8, 55.2)
- added R58: NC, Resistor_SMD:R_0402_1005Metric, F.Cu at (15.9, 56.9)
- added R59: 0R, Resistor_SMD:R_0402_1005Metric, F.Cu at (27.4, 44.9)
- added R60: NC, Resistor_SMD:R_0402_1005Metric, F.Cu at (15.9, 54.9)
- added U7: TPS5430DDA, Package_SO:TI_SO-PowerPAD-8_ThermalVias, F.Cu at (55.1, 47.2)
- C34: value 4.7u -> 0.1u
- C38: value 0.1u -> 220p
- J2, J5, J6, J7: footprint Connector_Molex:Molex_CLIK-Mate_502386-0370_1x03-1MP_P1.25mm_Horizontal -> Connector_PinHeader_2.54mm:PinHeader_1x03_P2.54mm_Vertical
- J3: value Conn_01x02 -> Conn_01x03; footprint Connector_PinHeader_2.54mm:PinHeader_1x02_P2.54mm_Vertical -> Connector_PinHeader_2.54mm:PinHeader_1x03_P2.54mm_Vertical
- J4: value USB_C_Receptacle -> Conn_01x03; footprint Connector_USB:USB_C_Receptacle_Palconn_UTC16-G -> Connector_PinHeader_2.54mm:PinHeader_1x03_P2.54mm_Vertical
- L1: value L -> 2.2uH
- M2: footprint ic_footprint:mini_elrs -> Connector_Molex:Molex_CLIK-Mate_502382-0470_1x04-1MP_P1.25mm_Vertical
- R14, R17: value 0R -> 100k
- R20: value 1.2k -> 0R
- R27: value 10K -> 100k
- R28: value 10K -> 100K
- U8: value ME6212C12M5G -> STM32F051K6Ux; footprint Package_TO_SOT_SMD:SOT-23-5 -> Package_DFN_QFN:QFN-32-1EP_5x5mm_P0.5mm_EP3.45x3.45mm; moved to F.Cu
- moved J4 40.7 mm to (101.6, 93.0), turned to 0 degrees
- moved J3 38.2 mm to (99.1, 98.0), turned to 180 degrees
- moved R17 33.2 mm to (63.2, 73.2)
- moved U8 30.7 mm to (96.0, 87.6), turned to 0 degrees
- moved R29 13.4 mm to (112.5, 80.3)
- moved M2 11.9 mm to (87.4, 49.8), turned to 0 degrees
- moved J5 11.3 mm to (88.9, 93.0)
- moved J2 10.3 mm to (86.1, 93.0)
- moved J7 9.49 mm to (91.4, 93.0)
- moved J6 7.96 mm to (83.6, 93.0)
Connections:
- net /U0_RX renamed /V3s_core/U0_RX
- net /U0_TX renamed /V3s_core/U0_TX
- C31 pad 1: +1V8 -> +1V2
- C34 pad 1: Net-(C34-Pad1) -> +1V2
- C38 pad 1: Net-(C34-Pad1) -> +1V2
- C38 pad 2: GND -> Net-(U3-Pad14)
- C56 pad 1: +1V8 -> GND
- C56 pad 2: GND -> /MCU_RST
- J2 pad 1: /FPGAIO5 -> /FPGAIO2
- J2 pad 2: +BATT -> +5VP
- J2 pad 3: Net-(Q1-Pad3) -> GNDPWR
- J3 pad 1: +BATT -> /FPGAIO0
- J3 pad 2: GNDPWR -> +5VP
- J5 pad 1: /FPGAIO1 -> /FPGAIO3
- J5 pad 2: +BATT -> +5VP
- J5 pad 3: Net-(Q2-Pad3) -> GNDPWR
- J6 pad 1: /FPGAIO7 -> /FPGAIO6
- J6 pad 2: +BATT -> +5VP
- J7 pad 1: /FPGAIO3 -> /FPGAIO4
- J7 pad 2: +BATT -> +5VP
- L1 pad 1: +BATT -> +1V2
- L1 pad 2: Net-(L1-Pad2) -> Net-(U3-Pad11)
- M1 pad 1: +1V8 -> +3V3
- M1 pad 10: /SD1_D3 -> /WIRQ
- M1 pad 11: (no net) -> /SD1_D3
- M1 pad 12: (no net) -> +1V8
- M1 pad 9: /WIRQ -> unconnected-(M1-Pad9)
- R14 pad 1: Net-(C34-Pad1) -> Net-(R14-Pad1)
- R14 pad 2: +1V2 -> +BATT
- R17 pad 2: GNDPWR -> Net-(R14-Pad1)
- R20 pad 1: Net-(R20-Pad1) -> GND
- R20 pad 2: GND -> GNDPWR
- R27 pad 1: Net-(D4-Pad2) -> GND
- R27 pad 2: Net-(R27-Pad2) -> Net-(U3-Pad14)
- R28 pad 1: /FPGAIO5 -> +1V2
- R28 pad 2: GNDPWR -> Net-(U3-Pad14)
- R29 pad 1: /FPGAIO1 -> GND
- R29 pad 2: GNDPWR -> Net-(R29-Pad2)
- U2 pad 32: unconnected-(U2-Pad32) -> /MCU_RST
- U2 pad 35: unconnected-(U2-Pad35) -> /V3s_core/CS_EXT1
- U2 pad 36: unconnected-(U2-Pad36) -> /V3s_core/CS_EXT2
- U3 pad 11: unconnected-(U3-Pad11) -> Net-(U3-Pad11)
- U3 pad 14: unconnected-(U3-Pad14) -> Net-(U3-Pad14)
- U8 pad 1: +1V8 -> +3.3V
- U8 pad 2: GND -> unconnected-(U8-Pad2)
- U8 pad 3: +1V8 -> unconnected-(U8-Pad3)
- U8 pad 4: unconnected-(U8-Pad4) -> /MCU_RST
- U8 pad 5: Net-(C34-Pad1) -> +3.3V
Routing:
- net GNDPWR: track 76.4 -> 0.00 mm, vias 13 -> 0
- net +5V: track 96.3 -> 20.9 mm, vias 6 -> 2
- net +BATT: track 65.9 -> 0.00 mm, vias 2 -> 0
- net /FPGAIO5: track 29.8 -> 0.00 mm, vias 3 -> 0
- net /FPGAIO7: track 27.3 -> 0.00 mm, vias 3 -> 0
- net /WIRQ: track 26.8 -> 0.00 mm, vias 2 -> 0
- net /SD1_D3: track 25.9 -> 0.00 mm, vias 1 -> 0
- net (no net): track 24.8 -> 0.00 mm
- net /FPGAIO1: track 22.9 -> 0.00 mm, vias 3 -> 0
- net VBUS: track 22.0 -> 0.00 mm
- net /U1_RX: track 20.8 -> 0.00 mm, vias 2 -> 0
- net /U1_TX: track 20.8 -> 0.00 mm, vias 2 -> 0
- net /USB_DN: track 20.4 -> 0.00 mm
- net /USB_DP: track 20.0 -> 0.00 mm
- net +1V8: track 87.0 -> 67.8 mm, vias 6 -> 4
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- removed copper zone on In1.Cu, net +3V3
- removed copper zone on B.Cu, net GND
- removed copper zone on F.Cu, net GND
