File: AutoPilotPi.kicad_sch (KiCad schematic)
At the start: 15 parts, among them J1 Conn_01x04_MountingPin, J4 USB_C_Receptacle, M1 xr819, M2 mini_elrs, U5 HMC5883L-TR, U6 SPL06-001

Commit message: v2.0-devel init
Signed-off-by: huangzzk <huangcmzzk@gmail.com>
Parts:
- removed J1: Conn_01x04_MountingPin, Connector_Molex:Molex_CLIK-Mate_502382-0470_1x04-1MP_P1.25mm_Vertical, symbol Connector_Generic_MountingPin:Conn_01x04_MountingPin
- removed J4: USB_C_Receptacle, Connector_USB:USB_C_Receptacle_Palconn_UTC16-G, symbol Connector:USB_C_Receptacle
- removed M1: xr819, ic_footprint:xr819_module, symbol modules:xr819
- removed M2: mini_elrs, ic_footprint:mini_elrs, symbol modules:mini_elrs
Other:
- added sheet AM32 (am32.kicad_sch)
- added sheet com (com.kicad_sch)
- sheet Power ports: added PWM5, PWM6, PWM7, PWM8; removed none
- moved on the sheet: C52, C53, C54, C55, I1, U6

Commit message: temply update
Signed-off-by: ncerzzk <huangzzk@bupt.edu.cn>
Parts:
- added J16, J17: Conn_01x04_MountingPin, Connector_Molex:Molex_CLIK-Mate_502382-0470_1x04-1MP_P1.25mm_Vertical, symbol Connector_Generic_MountingPin:Conn_01x04_MountingPin
- added J18: USB_C_Receptacle, Connector_USB:USB_C_Receptacle_Palconn_UTC16-G, symbol Connector:USB_C_Receptacle
- added J19: Conn_01x06_MountingPin, symbol Connector_Generic_MountingPin:Conn_01x06_MountingPin
- added M1: xr819, ic_footprint:xr819_module, symbol modules:xr819
- added M2: mini_elrs, Connector_Molex:Molex_CLIK-Mate_502382-0470_1x04-1MP_P1.25mm_Vertical, symbol modules:mini_elrs
- added R55, R57, R59: 0R, Resistor_SMD:R_0402_1005Metric, symbol Device:R
- added R56, R58, R60: NC, Resistor_SMD:R_0402_1005Metric, symbol Device:R
Connections:
- net +3V3: now also M1.1 (3V3), R56.2, R58.2, R60.2
- net GND: now also J18.A1 (GND), J18.A12 (GND), J18.B1 (GND), J18.B12 (GND), J18.S1 (SHIELD), M1.6 (GND), M2.4 (GND)
- net MISO: now also J19.4 (Pin_4)
- net MOSI: now also J19.3 (Pin_3)
- net SCL: now also J16.2 (Pin_2), J17.2 (Pin_2)
- net SCLK: now also J19.2 (Pin_2)
- net SD1_CLK: now also M1.7 (SCLK)
- net SD1_CMD: now also M1.8 (CMD)
- net SD1_D0: now also M1.5 (DATA0)
- net SD1_D1: now also M1.4 (DATA1)
- net SD1_D2: now also M1.3 (DATA2)
- net SD1_D3: now also M1.11 (DATA3)
- net SDA: now also J16.3 (Pin_3), J17.3 (Pin_3)
- net U1_RX: now also M2.3 (TX)
- net U1_TX: now also M2.2 (RX)
- net USB_DN: now also J18.A7 (D-), J18.B7 (D-)
- net USB_DP: now also J18.A6 (D+), J18.B6 (D+)
- net WIRQ: now also M1.10 (WIRQ)
- net WREST: now also M1.2 (RST)
- new net: R59.2, R60.1
- new net: J17.1 (Pin_1), R57.2, R58.1
- new net: J16.1 (Pin_1), R55.2, R56.1
- new net +1V8: M1.12 (1V8)
- new net +5V: M2.1 (5V)
- new net +5VP: R55.1, R57.1, R59.1
- new net CSN1: J19.5 (Pin_5)
- new net GNDPWR: J16.4 (Pin_4), J16.MP (MountPin), J17.4 (Pin_4), J17.MP (MountPin), J19.6 (Pin_6), J19.MP (MountPin)
- new net VBUS: J18.A4 (VBUS), J18.A9 (VBUS), J18.B4 (VBUS), J18.B9 (VBUS)
Other:
- removed sheet com
- sheet AM32 ports: added MISO, MOSI, NRST, NSS, PWM1, PWM2, PWM3, PWM4, PWM5, PWM6, PWM7, SCL, SCLK, SDA, U0RX, U0TX; removed none
- sheet V3s_core ports: added CS_EXT1, CS_EXT2, MCU_RST; removed U0_RX, U0_TX
- note added: "FPGA PIN Default:Weak pull up"
