File: AutoPilotPi.kicad_sch (KiCad schematic)
At the start: 15 parts, among them J1 Conn_01x04_MountingPin, J4 USB_C_Receptacle, M1 xr819, M2 mini_elrs, U5 HMC5883L-TR, U6 SPL06-001

Commit message: add esp32 as wifi card
Signed-off-by: huangzzk <huangcmzzk@gmail.com>
Parts:
- removed M1: xr819, ic_footprint:xr819_module, symbol modules:xr819
- removed M2: mini_elrs, ic_footprint:mini_elrs, symbol modules:mini_elrs
- added D5: D, Diode_SMD:D_0805_2012Metric, symbol Device:D
- added J9: Conn_01x04_MountingPin, Connector_Molex:Molex_CLIK-Mate_502382-0470_1x04-1MP_P1.25mm_Vertical, symbol Connector_Generic_MountingPin:Conn_01x04_MountingPin
Connections:
- net +5V: now also D5.2 (A), J9.1 (Pin_1)
- net GND: now also J9.4 (Pin_4), J9.MP (MountPin)
- net U1_RX: now also J9.3 (Pin_3)
- net U1_TX: now also J9.2 (Pin_2)
- net VBUS: now also D5.1 (K)
Other:
- added sheet esp32_wifi (esp32_wifi.kicad_sch)
- sheet V3s_core ports: added WLAN_ENABLE, WLAN_RESET2; removed WLAN_IRQ
