File: AutoPilotPi.kicad_sch (KiCad schematic)
At the start: 16 parts, among them J1 Conn_01x04_MountingPin, J2 Conn_01x04_MountingPin, J3 Conn_01x04_MountingPin, J4 USB_C_Receptacle, U5 HMC5883L-TR, U6 SPL06-001, U7 v3s_flight_controller

Commit message: use LDO to produce 1.2V, to fix fpga voltage issue. fix wrong fpga sch issue, change the pins of fpga. connect fpga SSPI to V3s-spi, so that we can configuare fpag on v3s someday.
Signed-off-by: ncerzzk <huangzzk@bupt.edu.cn>
Connections:
- net USB_ID: no longer J4.A8 (SBU1), J4.B8 (SBU2)
Other:
- sheet FPGA ports: added FPGA_CSN; removed FPGA_CTL0
Changed lines of the file:
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@@
-    (stroke (width 0) (type default) (color 0 0 0 0))
-  )
-  (wire (pts (xy 309.245 140.335) (xy 309.245 142.875))
     (stroke (width 0) (type default) (color 0 0 0 0))
   )
@@
   (label "SD1_D3" (at 132.715 40.005 180)
     (effects (font (size 1.27 1.27)) (justify right bottom))
-  )
-  (label "USB_ID" (at 309.245 140.335 0)
-    (effects (font (size 1.27 1.27)) (justify left bottom))
   )
   (label "MOSI" (at 164.465 75.565 0)
@@
       (effects (font (size 1.27 1.27)) (justify right))
     )
-    (pin "FPGA_CTL0" input (at 81.915 38.1 180)
-      (effects (font (size 1.27 1.27)) (justify left))
-    )
     (pin "TDI" input (at 109.855 62.865 0)
       (effects (font (size 1.27 1.27)) (justify right))
@@
     )
     (pin "SCLK" input (at 81.915 59.69 180)
+      (effects (font (size 1.27 1.27)) (justify left))
+    )
+    (pin "FPGA_CSN" input (at 81.915 38.1 180)
       (effects (font (size 1.27 1.27)) (justify left))
     )
@@
       (reference "#PWR029") (unit 1) (value "GND") (footprint "")
     )
+    (path "/2d8cbab5-6f7e-4d05-a82d-2f42b60a1429/04ece547-161e-455c-86b0-2f52b07ca91c"
+      (reference "#PWR030") (unit 1) (value "+5V") (footprint "")
+    )
+    (path "/2d8cbab5-6f7e-4d05-a82d-2f42b60a1429/3771ad80-761a-476c-bd5d-aecc56252d1c"
+      (reference "#PWR031") (unit 1) (value "GND") (footprint "")
+    )
+    (path "/2d8cbab5-6f7e-4d05-a82d-2f42b60a1429/67d8bdb5-20dd-4b89-8d0d-45a42b6dd4a2"
+      (reference "#PWR032") (unit 1) (value "+1V8") (footprint "")
+    )
+    (path "/2d8cbab5-6f7e-4d05-a82d-2f42b60a1429/d0b8745f-3f51-4beb-9b73-0afca456b537"
+      (reference "#PWR033") (unit 1) (value "GND") (footprint "")
+    )
+    (path "/2d8cbab5-6f7e-4d05-a82d-2f42b60a1429/e8b8e3eb-4813-4deb-a12a-706fe10a64de"
+      (reference "#PWR034") (unit 1) (value "GND") (footprint "")
+    )
+    (path "/2d8cbab5-6f7e-4d05-a82d-2f42b60a1429/65e597a8-b972-42f9-b5e6-5bb31c716891"
+      (reference "#PWR035") (unit 1) (value "GND") (footprint "")
+    )
+    (path "/2d8cbab5-6f7e-4d05-a82d-2f42b60a1429/4dbdcd7f-6393-44cf-a438-0209f867b181"
+      (reference "#PWR036") (unit 1) (value "+1V2") (footprint "")
+    )
     (path "/e76e4de2-72d1-495d-95b2-11c341ec23c6/231b371a-57c6-4c58-8631-8e9b67561612"
       (reference "#PWR0102") (unit 1) (value "+3V3") (footprint "")
@@
       (reference "#PWR0161") (unit 1) (value "+1V8") (footprint "")
     )
-    (path "/2d8cbab5-6f7e-4d05-a82d-2f42b60a1429/e4eda05d-47dc-4ebd-8028-e116d3c07a4e"
-      (reference "#PWR0162") (unit 1) (value "GND") (footprint "")
-    )
-    (path "/2d8cbab5-6f7e-4d05-a82d-2f42b60a1429/ebb07204-b3de-42c1-9519-fbf552c06002"
-      (reference "#PWR0163") (unit 1) (value "+1V2") (footprint "")
-    )
     (path "/2d8cbab5-6f7e-4d05-a82d-2f42b60a1429/a8290965-9531-4159-b92b-a6eeda9b32ba"
       (reference "#PWR0164") (unit 1) (value "VBUS") (footprint "")
@@
       (reference "#PWR0181") (unit 1) (value "+3V3") (footprint "")
     )
+    (path "/2d8cbab5-6f7e-4d05-a82d-2f42b60a1429/177ee29b-af28-4eea-bbb0-c132c1bed749"
+      (reference "1V2") (unit 1) (value "TestPoint") (footprint "TestPoint:TestPoint_Pad_1.0x1.0mm")
+    )
+    (path "/2d8cbab5-6f7e-4d05-a82d-2f42b60a1429/5e4cb721-104e-4bdd-9926-45e9d4291412"
+      (reference "1V8") (unit 1) (value "TestPoint") (footprint "TestPoint:TestPoint_Pad_1.0x1.0mm")
+    )
     (path "/e76e4de2-72d1-495d-95b2-11c341ec23c6/6794bc79-4b57-44b0-9037-eae2be66f87c"
       (reference "C1") (unit 1) (value "0.1u") (footprint "Capacitor_SMD:C_0402_1005Metric")
@@
       (reference "C30") (unit 1) (value "0.1u") (footprint "Capacitor_SMD:C_0402_1005Metric")
     )
-    (path "/2d8cbab5-6f7e-4d05-a82d-2f42b60a1429/e2896631-fade-4fb9-9dab-82dd679a77c0"
-      (reference "C31") (unit 1) (value "4.7u") (footprint "Capacitor_SMD:C_0402_1005Metric")
+    (path "/2d8cbab5-6f7e-4d05-a82d-2f42b60a1429/deee4f81-12be-4aee-b2c4-b743ad01f27f"
+      (reference "C31") (unit 1) (value "4.7uF") (footprint "Capacitor_SMD:C_0402_1005Metric")
     )
     (path "/2d8cbab5-6f7e-4d05-a82d-2f42b60a1429/895c8b0e-619d-4dcf-aa77-cf47de121dbf"
@@
       (reference "C33") (unit 1) (value "4.7u") (footprint "Capacitor_SMD:C_0402_1005Metric")
     )
-    (path "/2d8cbab5-6f7e-4d05-a82d-2f42b60a1429/55bcfc80-417c-45de-8d10-51fe4f4fee78"
-      (reference "C34") (unit 1) (value "0.1u") (footprint "Capacitor_SMD:C_0402_1005Metric")
+    (path "/2d8cbab5-6f7e-4d05-a82d-2f42b60a1429/f11a3a0e-1b0f-4c29-8b27-6c0990933767"
+      (reference "C34") (unit 1) (value "4.7uF") (footprint "Capacitor_SMD:C_0402_1005Metric")
     )
     (path "/2d8cbab5-6f7e-4d05-a82d-2f42b60a1429/3f3b66ea-042b-4e1e-bb22-d3f886de50c2"
@@
       (reference "C37") (unit 1) (value "220p") (footprint "Capacitor_SMD:C_0402_1005Metric")
     )
-    (path "/2d8cbab5-6f7e-4d05-a82d-2f42b60a1429/443c6915-3e7d-4dcc-a8f4-0007744c2520"
-      (reference "C38") (unit 1) (value "220p") (footprint "Capacitor_SMD:C_0402_1005Metric")
+    (path "/2d8cbab5-6f7e-4d05-a82d-2f42b60a1429/293f0b75-8e0d-40d7-b565-5ef2a151a0a5"
+      (reference "C38") (unit 1) (value "0.1u") (footprint "Capacitor_SMD:C_0402_1005Metric")
     )
     (path "/2d8cbab5-6f7e-4d05-a82d-2f42b60a1429/ee95c567-a5c0-4404-83c2-8db57014c312"
@@
       (reference "C55") (unit 1) (value "0.1u") (footprint "Capacitor_SMD:C_0402_1005Metric")
     )
+    (path "/2d8cbab5-6f7e-4d05-a82d-2f42b60a1429/8771269b-ed07-45d8-8ac8-443f861ab484"
+      (reference "C56") (unit 1) (value "0.1u") (footprint "Capacitor_SMD:C_0402_1005Metric")
+    )
     (path "/e76e4de2-72d1-495d-95b2-11c341ec23c6/ce1aa92b-84df-4f2b-b428-b8bdcefb805c"
       (reference "D1") (unit 1) (value "LED") (footprint "LED_SMD:LED_0603_1608Metric")
@@
       (reference "J4") (unit 1) (value "USB_C_Receptacle") (footprint "Connector_USB:USB_C_Receptacle_Palconn_UTC16-G")
     )
-    (path "/2d8cbab5-6f7e-4d05-a82d-2f42b60a1429/6150f233-d4a0-4b18-839d-1ddb5e6b1e8f"
-      (reference "L1") (unit 1) (value "2.2uH") (footprint "Inductor_SMD:L_Abracon_ASPI-3012S")
-    )
     (path "/2d8cbab5-6f7e-4d05-a82d-2f42b60a1429/c9898a43-521f-4634-b755-376115d5aa6f"
       (reference "L2") (unit 1) (value "2.2uH") (footprint "Inductor_SMD:L_Abracon_ASPI-3012S")
@@
       (reference "R13") (unit 1) (value "NC") (footprint "Resistor_SMD:R_0402_1005Metric")
     )
-    (path "/2d8cbab5-6f7e-4d05-a82d-2f42b60a1429/1743fe4f-bea3-4579-acee-c147ec8b9ced"
-      (reference "R14") (unit 1) (value "100k") (footprint "Resistor_SMD:R_0402_1005Metric")
+    (path "/2d8cbab5-6f7e-4d05-a82d-2f42b60a1429/08b59541-918b-45c0-89d5-5c3dff09356f"
+      (reference "R14") (unit 1) (value "0R") (footprint "Resistor_SMD:R_0402_1005Metric")
     )
     (path "/2d8cbab5-6f7e-4d05-a82d-2f42b60a1429/1f662fb7-291e-4cca-99ff-5246b31c7542"
@@
       (reference "R16") (unit 1) (value "100k") (footprint "Resistor_SMD:R_0402_1005Metric")
     )
-    (path "/2d8cbab5-6f7e-4d05-a82d-2f42b60a1429/e8e6d1af-95fe-4d93-922e-e5501e366c90"
-      (reference "R17") (unit 1) (value "100k") (footprint "Resistor_SMD:R_0402_1005Metric")
-    )
     (path "/2d8cbab5-6f7e-4d05-a82d-2f42b60a1429/d1b36604-bafc-4e63-9d45-d69e82aff9be"
       (reference "R18") (unit 1) (value "680k") (footprint "Resistor_SMD:R_0402_1005Metric")
@@
     )
     (path "/46301cab-1d7b-4022-921a-2b4b16934078/c838c6ae-f4b4-4703-b9b9-6a89bb9f90b1"
-      (reference "R21") (unit 1) (value "10K") (footprint "Resistor_SMD:R_0402_1005Metric")
+      (reference "R21") (unit 1) (value "0R") (footprint "Resistor_SMD:R_0402_1005Metric")
     )
     (path "/e1ae0837-2279-4998-943a-7864ce3e1f0f"
@@
       (reference "SW1") (unit 1) (value "SW_Push") (footprint "Button_Switch_SMD:SW_Push_SPST_NO_Alps_SKRK")
     )
-    (path "/2d8cbab5-6f7e-4d05-a82d-2f42b60a1429/5e4cb721-104e-4bdd-9926-45e9d4291412"
-      (reference "TP1") (unit 1) (value "TestPoint") (footprint "TestPoint:TestPoint_Pad_1.0x1.0mm")
-    )
-    (path "/2d8cbab5-6f7e-4d05-a82d-2f42b60a1429/177ee29b-af28-4eea-bbb0-c132c1bed749"
-      (reference "TP2") (unit 1) (value "TestPoint") (footprint "TestPoint:TestPoint_Pad_1.0x1.0mm")
-    )
     (path "/e76e4de2-72d1-495d-95b2-11c341ec23c6/e1f2697a-633a-4c4c-8f2e-b6746633c3b2"
       (reference "U1") (unit 1) (value "MKDV4GCL-AB") (footprint "ic_footprint:LGA-8_L8.0-W6.0-BL_MKDV4GIL-AS")
@@
       (reference "U7") (unit 1) (value "v3s_flight_controller") (footprint "ic_footprint:Flight_Core")
     )
+    (path "/2d8cbab5-6f7e-4d05-a82d-2f42b60a1429/a86ad215-93f2-430d-a55b-dc700351bc4e"
+      (reference "U8") (unit 1) (value "TLV71312PDBV") (footprint "Package_TO_SOT_SMD:SOT-23-5")
+    )
     (path "/e76e4de2-72d1-495d-95b2-11c341ec23c6/470675a5-f091-41b7-ad3e-a3f31dce5b8f"
       (reference "Y1") (unit 1) (value "Crystal") (footprint "Crystal:Crystal_SMD_3215-2Pin_3.2x1.5mm")
     )
     (path "/e76e4de2-72d1-495d-95b2-11c341ec23c6/6d13e815-134d-4772-b8f1-a65402700c45"
-      (reference "Y2") (unit 1) (value "Crystal_GND24_Small") (footprint "Crystal:Crystal_SMD_EuroQuartz_MT-4Pin_3.2x2.5mm_HandSoldering")
-    )
-  )
+      (reference "Y2") (unit 1) (value "Crystal_GND24_Small") (footprint "Crystal:Crystal_SMD_EuroQuartz_MT-4Pin_3.2x2.5mm")
+    )
+  )

Commit message: update 2.0
Signed-off-by: huangzzk <huangcmzzk@gmail.com>
Connections:
- net FPGA/TCK: no longer U7.12 (TCK)
- net FPGA/TDI: no longer U7.11 (TDI)
- net FPGA/TDO: no longer U7.10 (TDO)
- net FPGA/TMS: no longer U7.13 (TMS)
- net FPGAIO7: now also U7.13 (IO7)
- net USB_DN: now also U7.11 (USB_DN)
- net USB_DP: now also U7.10 (USB_DP)
- net CSN renamed USER_CSN1
- new net GPIO_EXT0: U7.38 (EXT0)
- new net GPIO_EXT1: U7.39 (EXT1)
- new net GPIO_EXT10: U7.45 (EXT7)
- new net GPIO_EXT11: U7.35 (EXT11)
- new net GPIO_EXT12: U7.36 (EXT12)
- new net GPIO_EXT13: U7.37 (EXT13)
- new net GPIO_EXT2: U7.40 (EXT2)
- new net GPIO_EXT3: U7.44 (EXT6)
- new net GPIO_EXT4: U7.48 (EXT10)
- new net GPIO_EXT5: U7.43 (EXT5)
- new net GPIO_EXT6: U7.47 (EXT9)
- new net GPIO_EXT7: U7.42 (EXT4)
- new net GPIO_EXT8: U7.46 (EXT8)
- new net GPIO_EXT9: U7.41 (EXT3)
- new net USER_CSN2: U7.12 (CSN2)
Other:
- sheet FPGA ports: added PLL_IN; removed none
- sheet V3s_core ports: added GPIO_EXT0, GPIO_EXT1, GPIO_EXT10, GPIO_EXT11, GPIO_EXT12, GPIO_EXT13, GPIO_EXT2, GPIO_EXT3, GPIO_EXT4, GPIO_EXT5, GPIO_EXT6, GPIO_EXT7, GPIO_EXT8, GPIO_EXT9, PWM_OUT, USER_CS1, USER_CSN2; removed CS
- note added: "You can also use: ICM20688 QMI8658A ..."
- note removed: "Replace FPGAIO7 by CS(V3s) Out. To make the users use spi directly."
