File: V3s_core.kicad_sch (KiCad schematic)
At the start: 55 parts, among them SW1 SW_Push, U1 MKDV4GCL-AB, U2 V3S-ALLWINNER, Y1 Crystal, Y2 Crystal_GND24_Small

Commit message: update mini
Signed-off-by: huangzzk <huangcmzzk@gmail.com>
Parts:
- removed R27: 499R, Resistor_SMD:R_0402_1005Metric, symbol Device:R
- removed SW1: SW_Push, Button_Switch_SMD:SW_Push_SPST_NO_Alps_SKRK, symbol Switch:SW_Push
- C11, C12, C17, C18: value 18pf -> 18p
- C15: value 1uF -> 1u
Connections:
- net WLAN_IRQ: now reaches U2.6 (PE24/LCD_D23)
- net WLAN_REST: now reaches U2.7 (PE23/LCD_D22)

Commit message: v2.0-devel init
Signed-off-by: huangzzk <huangcmzzk@gmail.com>
Other:
- moved on the sheet: C1, D1, D2, D3, R24, R25, R26, U1, U2K

Commit message: temply update
Signed-off-by: ncerzzk <huangzzk@bupt.edu.cn>
Parts:
- added J1: Conn_01x04_MountingPin, Connector_Molex:Molex_CLIK-Mate_502382-0470_1x04-1MP_P1.25mm_Vertical, symbol Connector_Generic_MountingPin:Conn_01x04_MountingPin
Connections:
- net GND: now also J1.4 (Pin_4), J1.MP (MountPin)
- net U0_RX: now also J1.3 (Pin_3)
- net U0_TX: now also J1.2 (Pin_2)
- net MCU_RST: now reaches U2.32 (PE5/CSI_D1/LCD_D3)
- net CS_EXT1: now reaches U2.35 (PE2/CSI_HSYNC/LCD_HSYNC)
- net CS_EXT2: now reaches U2.36 (PE1/CSI_MCLK/LCD_DE)
- new net +5V: J1.1 (Pin_1)
Other:
- moved on the sheet: C3
