File: V3s_core.kicad_sch (KiCad schematic)
At the start: 53 parts, among them U1 MKDV4GCL-AB, U2 V3S-ALLWINNER, Y1 Crystal, Y2 Crystal_GND24_Small

Commit message: add esp32 as wifi card
Signed-off-by: huangzzk <huangcmzzk@gmail.com>
Connections:
- net WLAN_RESET2: now reaches U2.10 (PE20/CSI_FIELD/CSI_MIPI_MCLK)
- net WLAN_IRQ renamed WLAN_ENABLE
Changed lines of the file:
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@@
+    (effects (font (size 1.27 1.27)) (justify right))
+  )
+  (hierarchical_label "WLAN_RESET2" (shape input) (at 120.015 48.26 180)
     (effects (font (size 1.27 1.27)) (justify right))
   )
@@
     (effects (font (size 1.27 1.27)) (justify right))
   )
-  (hierarchical_label "WLAN_IRQ" (shape input) (at 120.015 38.1 180)
+  (hierarchical_label "WLAN_ENABLE" (shape input) (at 120.015 38.1 180)
     (effects (font (size 1.27 1.27)) (justify right))
   )
