File: am32.kicad_sch (KiCad schematic)
At the start: 1 part

Commit message: temply update
Signed-off-by: huangzzk <huangcmzzk@gmail.com>
Parts:
- added C?: 0.1u, Capacitor_SMD:C_0402_1005Metric, symbol Device:C
- added J?: Conn_01x03, symbol Connector_Generic:Conn_01x03
- added R? (x2): 10K, Resistor_SMD:R_0402_1005Metric, symbol Device:R
Connections:
- net +3.3V: now also J?.1 (Pin_1), R?.2
- net GND: now also C?.1, J?.3 (Pin_3), R?.1
- net at U?.31 (BOOT0): now also R?.2
- net at U?.4 (NRST): now also C?.2, R?.1
- new net ADC1: J?.2 (Pin_2)

Commit message: temply update
Signed-off-by: ncerzzk <huangzzk@bupt.edu.cn>
Parts:
- added J10, J12, J13, J14, J15: Conn_01x03, Connector_Molex:Molex_PicoBlade_53047-0310_1x03_P1.25mm_Vertical, symbol Connector_Generic:Conn_01x03
- added R31, R32, R35, R36, R39, R40, R42, R44, R47, R48, R51, R52: 0R, Resistor_SMD:R_0402_1005Metric, symbol Device:R
- added R33, R34, R37, R38, R41, R43, R45, R46, R49, R50, R53, R54: NC, Resistor_SMD:R_0402_1005Metric, symbol Device:R
- J11: renamed from J?; footprint (none) -> Connector_Molex:Molex_PicoBlade_53047-0310_1x03_P1.25mm_Vertical
- gave numbers to parts that had none: 4
Connections:
- net +3.3V: now also R31.2, R35.2, R39.2, R42.2, R47.2, R51.2; no longer J11.1 (Pin_1)
- net ADC1: now also U8.7 (PA1), R36.1, R37.2; no longer J11.2 (Pin_2)
- net GND: now also J10.3 (Pin_3), J12.3 (Pin_3), J13.3 (Pin_3), J14.3 (Pin_3), J15.3 (Pin_3), R33.1, R37.1, R41.1, R45.1, R49.1, R53.1
- net NRST: now reaches C56.2, R30.1, U8.4 (NRST)
- net ADC4: now reaches U8.10 (PA4)
- net ADC4: now also R52.1, R53.2
- net ADC5: now reaches U8.11 (PA5)
- net ADC5: now also R40.1, R41.2
- net MISO: now reaches U8.12 (PA6)
- net MOSI: now reaches U8.13 (PA7)
- net PWM3: now reaches U8.14 (PB0)
- net PWM4: now reaches U8.15 (PB1)
- net PWM1: now reaches U8.18 (PA8)
- net U0TX: now reaches U8.19 (PA9)
- net U0RX: now reaches U8.20 (PA10)
- net PWM2: now reaches U8.21 (PA11)
- net SWDIO: now reaches U8.23 (PA13)
- net SWCLK: now reaches U8.24 (PA14)
- net NSS: now reaches U8.25 (PA15)
- net SCLK: now reaches U8.26 (PB3)
- net PWM5: now reaches U8.27 (PB4)
- net PWM6: now reaches U8.28 (PB5)
- net SCL: now reaches U8.29 (PB6)
- net SDA: now reaches U8.30 (PB7)
- net PWM7: now reaches U8.32 (PB8)
- net ADC0: now reaches U8.6 (PA0)
- net ADC0: now also R32.1, R33.2
- net ADC2: now reaches U8.8 (PA2)
- net ADC2: now also R44.1, R45.2
- net ADC3: now reaches U8.9 (PA3)
- net ADC3: now also R48.1, R49.2
- new net: J14.1 (Pin_1), R47.1, R50.1
- new net: J13.1 (Pin_1), R42.1, R46.1
- new net: J11.1 (Pin_1), R35.1, R38.1
- new net: J11.2 (Pin_2), R36.2
- new net: J15.1 (Pin_1), R51.1, R54.1
- new net: J10.1 (Pin_1), R31.1, R34.1
- new net: J10.2 (Pin_2), R32.2
- new net: J12.1 (Pin_1), R39.1, R43.1
- new net: J14.2 (Pin_2), R48.2
- new net: J13.2 (Pin_2), R44.2
- new net: J12.2 (Pin_2), R40.2
- new net: J15.2 (Pin_2), R52.2
- new net +5V: R34.2, R38.2, R43.2, R46.2, R50.2, R54.2
Other:
- moved on the sheet: J11, R30
