File: com.kicad_sch (KiCad schematic)
At the start: 13 parts

Commit message: temply update
Signed-off-by: ncerzzk <huangzzk@bupt.edu.cn>
Parts:
- removed J?: Conn_01x06_MountingPin, symbol Connector_Generic_MountingPin:Conn_01x06_MountingPin
- removed J? (x3): Conn_01x04_MountingPin, Connector_Molex:Molex_CLIK-Mate_502382-0470_1x04-1MP_P1.25mm_Vertical, symbol Connector_Generic_MountingPin:Conn_01x04_MountingPin
- removed J?: USB_C_Receptacle, Connector_USB:USB_C_Receptacle_Palconn_UTC16-G, symbol Connector:USB_C_Receptacle
- removed M?: xr819, ic_footprint:xr819_module, symbol modules:xr819
- removed M?: mini_elrs, ic_footprint:mini_elrs, symbol modules:mini_elrs
- removed R? (x3): NC, Resistor_SMD:R_0402_1005Metric, symbol Device:R
- removed R? (x3): 0R, Resistor_SMD:R_0402_1005Metric, symbol Device:R
