File: power.kicad_sch (KiCad schematic)
At the start: 36 parts, among them U3 EA3036

Commit message: temply update
Signed-off-by: ncerzzk <huangzzk@bupt.edu.cn>
Parts:
- added R20: 0R, Resistor_SMD:R_0402_1005Metric, symbol Device:R
- J2, J3, J4, J5, J6, J7, J8, J9: renamed from J?; footprint (none) -> Connector_PinHeader_2.54mm:PinHeader_1x03_P2.54mm_Vertical
- gave numbers to parts that had none: 9
Connections:
- net GND: now also R20.1
- net GNDPWR: now also R20.2
