File: FPGA.kicad_sch (KiCad schematic)
At the start: 8 parts, among them U4 GW1N_LV4QN32C6/I5

Commit message: update 2.0
Signed-off-by: huangzzk <huangcmzzk@gmail.com>
Parts:
- R21: value 0R -> NC
Connections:
- net +3V3: no longer U4.15 (IOR4A/RPLL_T_fb)
- net FPGAIO9: now also U4.15 (IOR4A/RPLL_T_fb); no longer U4.14 (IOR5A/GCLKT_2/RPLL_T_in)
- new net PLL_IN: U4.14 (IOR5A/GCLKT_2/RPLL_T_in)
Other:
- note added: "GW1N-1 IOL6 IOR6 don't support I/O"
Changed lines of the file:
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@@
+    (stroke (width 0) (type default) (color 0 0 0 0))
+  )
+  (wire (pts (xy 85.725 92.075) (xy 95.885 92.075))
     (stroke (width 0) (type default) (color 0 0 0 0))
   )
@@
     (stroke (width 0) (type default) (color 0 0 0 0))
   )
-  (wire (pts (xy 87.63 94.615) (xy 95.885 94.615))
-    (stroke (width 0) (type default) (color 0 0 0 0))
-  )
   (wire (pts (xy 162.56 94.615) (xy 154.305 94.615))
     (stroke (width 0) (type default) (color 0 0 0 0))
@@
     (stroke (width 0) (type default) (color 0 0 0 0))
   )
+  (text "GW1N-1 IOL6 IOR6 don't support I/O" (at 81.28 113.03 0)
+    (effects (font (size 1.27 1.27)) (justify left bottom))
+  )
   (hierarchical_label "SDA" (shape input) (at 154.305 66.675 0)
     (effects (font (size 1.27 1.27)) (justify left))
@@
     (effects (font (size 1.27 1.27)) (justify right))
   )
+  (hierarchical_label "FPGAIO9" (shape bidirectional) (at 95.885 94.615 180)
+    (effects (font (size 1.27 1.27)) (justify right))
+  )
   (hierarchical_label "FPGAIO6" (shape bidirectional) (at 154.305 64.135 0)
     (effects (font (size 1.27 1.27)) (justify left))
@@
     (effects (font (size 1.27 1.27)) (justify left))
   )
-  (hierarchical_label "FPGAIO9" (shape bidirectional) (at 95.885 92.075 180)
+  (hierarchical_label "PLL_IN" (shape bidirectional) (at 85.725 92.075 180)
     (effects (font (size 1.27 1.27)) (justify right))
   )
@@
   (hierarchical_label "TDI" (shape input) (at 154.305 84.455 0)
     (effects (font (size 1.27 1.27)) (justify left))
-  )
-  (symbol (lib_id "power:+3V3") (at 87.63 94.615 90) (unit 1)
-    (in_bom yes) (on_board yes)
-    (property "Reference" "#PWR0169" (id 0) (at 91.44 94.615 0)
-      (effects (font (size 1.27 1.27)) hide)
-    )
-    (property "Value" "+3V3" (id 1) (at 86.995 93.98 90)
-      (effects (font (size 1.27 1.27)) (justify right))
-    )
-    (property "Footprint" "" (id 2) (at 87.63 94.615 0)
-      (effects (font (size 1.27 1.27)) hide)
-    )
-    (property "Datasheet" "" (id 3) (at 87.63 94.615 0)
-      (effects (font (size 1.27 1.27)) hide)
-    )
-    (pin "1")
   )
   (symbol (lib_id "power:+3V3") (at 39.37 65.405 0) (unit 1)
@@
     (in_bom yes) (on_board yes)
     (property "Reference" "R21" (id 0) (at 161.925 66.675 90))
-    (property "Value" "0R" (id 1) (at 164.465 69.85 90))
+    (property "Value" "NC" (id 1) (at 164.465 69.85 90))
     (property "Footprint" "Resistor_SMD:R_0402_1005Metric" (id 2) (at 162.56 73.533 90)
       (effects (font (size 1.27 1.27)) hide)
